Commit message: v5

File: install/my_pib_description/share/my_pib_description/urdf/robot.urdf (robot description, URDF)
Before this commit: robot pib, 39 links, 38 joints
Links:
- removed link urdf_elbow-lower
- removed link urdf_elbow-upper
- removed link urdf_finger_distal
- removed link urdf_finger_distal_10
- removed link urdf_finger_distal_2
- removed link urdf_finger_distal_3
- removed link urdf_finger_distal_4
- removed link urdf_finger_distal_5
- removed link urdf_finger_distal_6
- removed link urdf_finger_distal_7
- removed link urdf_finger_distal_8
- removed link urdf_finger_distal_9
- removed link urdf_finger_proximal
- removed link urdf_finger_proximal_10
- removed link urdf_finger_proximal_2
- removed link urdf_finger_proximal_3
- removed link urdf_finger_proximal_4
- removed link urdf_finger_proximal_5
- removed link urdf_finger_proximal_6
- removed link urdf_finger_proximal_7
- removed link urdf_finger_proximal_8
- removed link urdf_finger_proximal_9
- removed link urdf_forearm
- removed link urdf_palm_left
- removed link urdf_palm_right
- removed link urdf_shoulder_horizontal
- removed link urdf_shoulder_vertical
- removed link urdf_thumb_rotator_left
- removed link urdf_thumb_rotator_right
Joints:
- removed joint elbow_left
- removed joint forearm_left
- removed joint index_left_distal
- removed joint index_left_proximal
- removed joint index_right_distal
- removed joint index_right_proximal
- removed joint middle_left_distal
- removed joint middle_left_proximal
- removed joint middle_right_distal
- removed joint middle_right_proximal
- removed joint pinky_left_distal
- removed joint pinky_left_proximal
- removed joint pinky_right_distal
- removed joint pinky_right_proximal
- removed joint ring_left_distal
- removed joint ring_left_proximal
- removed joint ring_right_distal
- removed joint ring_right_proximal
- removed joint shoulder_horizontal_left
- removed joint shoulder_vertical_left
- removed joint thumb_left_distal
- removed joint thumb_left_opposition
- removed joint thumb_left_proximal
- removed joint thumb_right_distal
- removed joint thumb_right_opposition
- removed joint thumb_right_proximal
- removed joint upper_arm_left
- removed joint wrist_left
- removed joint wrist_right
- joint base_link_to_base: origin xyz=0 0 0 rpy=0.0 0 0 -> xyz=0 0 -0.35 rpy=0.0 0 0

File: src/my_pib_description/urdf/robot.urdf (robot description, URDF)
Before this commit: robot pib, 10 links, 9 joints
Joints:
- joint base_link_to_base: origin xyz=0 0 0 rpy=0.0 0 0 -> xyz=0 0 -0.35 rpy=0.0 0 0

Commit message: v6

File: install/my_pib_description/share/my_pib_description/urdf/robot.urdf (robot description, URDF)
Before this commit: robot pib, 10 links, 9 joints
Links:
- removed link urdf_camera_link
Joints:
- removed joint camera

Commit message: v8

File: install/my_pib_description/share/my_pib_description/urdf/robot.urdf (robot description, URDF)
Before this commit: robot pib, 9 links, 8 joints
Links:
- added link tool_link
- link urdf_body: geometry collision mesh filename=package://my_pib_description/meshes/urdf_body1.stl; visual mesh filename=package://my_pib_description/meshes/urdf_body1.stl
Joints:
- added joint tool_joint: type fixed, parent urdf_forearm_2, child tool_link, origin xyz=0 0 0 rpy=0 0 0

Commit message: v9

File: install/my_pib_description/share/my_pib_description/urdf/robot.urdf (robot description, URDF)
Before this commit: robot pib, 10 links, 9 joints
Links:
- removed link tool_link
Joints:
- removed joint tool_joint

File: src/my_pib_description/urdf/robot.urdf (robot description, URDF)
Before this commit: robot pib, 10 links, 9 joints
Links:
- link tool_link: mass None -> 0.001

Commit message: v10

File: install/my_pib_description/share/my_pib_description/urdf/robot.urdf (robot description, URDF)
Before this commit: robot pib, 9 links, 8 joints
Links:
- added link tool_link, mass 0.001
- link urdf_body: geometry collision mesh filename=package://my_pib_description/meshes/urdf_body.stl; visual mesh filename=package://my_pib_description/meshes/urdf_body.stl
Joints:
- added joint tool_joint: type fixed, parent urdf_forearm_2, child tool_link, origin xyz=0 0 0 rpy=0 0 0

File: src/my_pib_description/urdf/robot.urdf (robot description, URDF)
Before this commit: robot pib, 10 links, 9 joints
Links:
- link urdf_body: geometry collision mesh filename=package://my_pib_description/meshes/urdf_body.stl; visual mesh filename=package://my_pib_description/meshes/urdf_body.stl
