Commit message: v4

File: src/my_pib_description/urdf/robot.urdf (robot description, URDF)
Before this commit: robot pib, 39 links, 38 joints
Links:
- removed link urdf_elbow-lower
- removed link urdf_elbow-upper
- removed link urdf_finger_distal
- removed link urdf_finger_distal_10
- removed link urdf_finger_distal_2
- removed link urdf_finger_distal_3
- removed link urdf_finger_distal_4
- removed link urdf_finger_distal_5
- removed link urdf_finger_distal_6
- removed link urdf_finger_distal_7
- removed link urdf_finger_distal_8
- removed link urdf_finger_distal_9
- removed link urdf_finger_proximal
- removed link urdf_finger_proximal_10
- removed link urdf_finger_proximal_2
- removed link urdf_finger_proximal_3
- removed link urdf_finger_proximal_4
- removed link urdf_finger_proximal_5
- removed link urdf_finger_proximal_6
- removed link urdf_finger_proximal_7
- removed link urdf_finger_proximal_8
- removed link urdf_finger_proximal_9
- removed link urdf_forearm
- removed link urdf_palm_left
- removed link urdf_palm_right
- removed link urdf_shoulder_horizontal
- removed link urdf_shoulder_vertical
- removed link urdf_thumb_rotator_left
- removed link urdf_thumb_rotator_right
Joints:
- removed joint elbow_left
- removed joint forearm_left
- removed joint index_left_distal
- removed joint index_left_proximal
- removed joint index_right_distal
- removed joint index_right_proximal
- removed joint middle_left_distal
- removed joint middle_left_proximal
- removed joint middle_right_distal
- removed joint middle_right_proximal
- removed joint pinky_left_distal
- removed joint pinky_left_proximal
- removed joint pinky_right_distal
- removed joint pinky_right_proximal
- removed joint ring_left_distal
- removed joint ring_left_proximal
- removed joint ring_right_distal
- removed joint ring_right_proximal
- removed joint shoulder_horizontal_left
- removed joint shoulder_vertical_left
- removed joint thumb_left_distal
- removed joint thumb_left_opposition
- removed joint thumb_left_proximal
- removed joint thumb_right_distal
- removed joint thumb_right_opposition
- removed joint thumb_right_proximal
- removed joint upper_arm_left
- removed joint wrist_left
- removed joint wrist_right

Commit message: v15

File: src/my_pib_description/urdf/robot.urdf (robot description, URDF)
Before this commit: robot pib, 10 links, 9 joints
Joints:
- joint tool_joint: origin xyz=0 0 0 rpy=0 0 0 -> xyz=0 0 -0.14 rpy=0 0 0

File: src/pib_moveit_config/config/pib.ros2_control.xacro (robot description, xacro)
@@ -8,16 +8,4 @@
                 <plugin>mock_components/GenericSystem</plugin>
             </hardware>
-            <joint name="head_horizontal">
-                <command_interface name="position"/>
-                <state_interface name="position">
-                  <param name="initial_value">${initial_positions['head_horizontal']}</param>
-                </state_interface>
-            </joint>
-            <joint name="head_vertical">
-                <command_interface name="position"/>
-                <state_interface name="position">
-                  <param name="initial_value">${initial_positions['head_vertical']}</param>
-                </state_interface>
-            </joint>
             <joint name="shoulder_vertical_right">
                 <command_interface name="position"/>
